File: diyperksmic.sch (KiCad schematic (older format))
At the start: 22 parts, among them J1 Conn_01x03, J2 Conn_Coaxial, J3 Conn_01x02, J4 Conn_01x02, Q1 Q_NJFET_GDS, U1 THAT1512, U2 NMA0515SC

Commit message: updated kicad board
fix resistor sizes and cap sizes
Parts:
- C1, C2, C5: footprint Capacitor_THT:CP_Radial_D5.0mm_P2.50mm -> Capacitor_THT:C_Disc_D8.0mm_W5.0mm_P5.00mm
- R1: footprint Resistor_THT:R_Axial_DIN0309_L9.0mm_D3.2mm_P12.70mm_Horizontal -> Resistor_THT:R_Axial_DIN0207_L6.3mm_D2.5mm_P10.16mm_Horizontal
- R2, R3, R4, R5, R6, R7, R8: footprint Resistor_THT:R_Axial_DIN0309_L9.0mm_D3.2mm_P15.24mm_Horizontal -> Resistor_THT:R_Axial_DIN0207_L6.3mm_D2.5mm_P10.16mm_Horizontal
Changed lines of the file:
@@
 F 0 "R1" H 2320 3246 50  0000 L CNN
 F 1 "2.2K" H 2320 3155 50  0000 L CNN
-F 2 "Resistor_THT:R_Axial_DIN0309_L9.0mm_D3.2mm_P12.70mm_Horizontal" V 2180 3200 50  0001 C CNN
+F 2 "Resistor_THT:R_Axial_DIN0207_L6.3mm_D2.5mm_P10.16mm_Horizontal" V 2180 3200 50  0001 C CNN
 F 3 "~" H 2250 3200 50  0001 C CNN
 	1    2250 3200
@@
 F 0 "R5" H 4470 3796 50  0000 L CNN
 F 1 "3.9K" H 4470 3705 50  0000 L CNN
-F 2 "Resistor_THT:R_Axial_DIN0309_L9.0mm_D3.2mm_P15.24mm_Horizontal" V 4330 3750 50  0001 C CNN
+F 2 "Resistor_THT:R_Axial_DIN0207_L6.3mm_D2.5mm_P10.16mm_Horizontal" V 4330 3750 50  0001 C CNN
 F 3 "~" H 4400 3750 50  0001 C CNN
 	1    4400 3750
@@
 F 0 "R2" H 2320 4696 50  0000 L CNN
 F 1 "2.2K" H 2320 4605 50  0000 L CNN
-F 2 "Resistor_THT:R_Axial_DIN0309_L9.0mm_D3.2mm_P15.24mm_Horizontal" V 2180 4650 50  0001 C CNN
+F 2 "Resistor_THT:R_Axial_DIN0207_L6.3mm_D2.5mm_P10.16mm_Horizontal" V 2180 4650 50  0001 C CNN
 F 3 "~" H 2250 4650 50  0001 C CNN
 	1    2250 4650
@@
 F 0 "R3" H 5470 3046 50  0000 L CNN
 F 1 "2.2K" H 5470 2955 50  0000 L CNN
-F 2 "Resistor_THT:R_Axial_DIN0309_L9.0mm_D3.2mm_P15.24mm_Horizontal" V 5330 3000 50  0001 C CNN
+F 2 "Resistor_THT:R_Axial_DIN0207_L6.3mm_D2.5mm_P10.16mm_Horizontal" V 5330 3000 50  0001 C CNN
 F 3 "~" H 5400 3000 50  0001 C CNN
 	1    5400 3000
@@
 F 0 "R4" H 6370 5346 50  0000 L CNN
 F 1 "2.2K" H 6370 5255 50  0000 L CNN
-F 2 "Resistor_THT:R_Axial_DIN0309_L9.0mm_D3.2mm_P15.24mm_Horizontal" V 6230 5300 50  0001 C CNN
+F 2 "Resistor_THT:R_Axial_DIN0207_L6.3mm_D2.5mm_P10.16mm_Horizontal" V 6230 5300 50  0001 C CNN
 F 3 "~" H 6300 5300 50  0001 C CNN
 	1    6300 5300
@@
 F 0 "R6" H 4170 4496 50  0000 L CNN
 F 1 "3.9K" H 4170 4405 50  0000 L CNN
-F 2 "Resistor_THT:R_Axial_DIN0309_L9.0mm_D3.2mm_P15.24mm_Horizontal" V 4030 4450 50  0001 C CNN
+F 2 "Resistor_THT:R_Axial_DIN0207_L6.3mm_D2.5mm_P10.16mm_Horizontal" V 4030 4450 50  0001 C CNN
 F 3 "~" H 4100 4450 50  0001 C CNN
 	1    4100 4450
@@
 F 0 "C2" V 2948 4150 50  0000 C CNN
 F 1 "22uF" V 3039 4150 50  0000 C CNN
-F 2 "Capacitor_THT:CP_Radial_D5.0mm_P2.50mm" H 3238 4000 50  0001 C CNN
+F 2 "Capacitor_THT:C_Disc_D8.0mm_W5.0mm_P5.00mm" H 3238 4000 50  0001 C CNN
 F 3 "~" H 3200 4150 50  0001 C CNN
 	1    3200 4150
@@
 F 0 "C1" V 2948 3450 50  0000 C CNN
 F 1 "22uF" V 3039 3450 50  0000 C CNN
-F 2 "Capacitor_THT:CP_Radial_D5.0mm_P2.50mm" H 3238 3300 50  0001 C CNN
+F 2 "Capacitor_THT:C_Disc_D8.0mm_W5.0mm_P5.00mm" H 3238 3300 50  0001 C CNN
 F 3 "~" H 3200 3450 50  0001 C CNN
 	1    3200 3450
@@
 F 0 "C5" V 7698 3750 50  0000 C CNN
 F 1 "22uF" V 7789 3750 50  0000 C CNN
-F 2 "Capacitor_THT:CP_Radial_D5.0mm_P2.50mm" H 7988 3600 50  0001 C CNN
+F 2 "Capacitor_THT:C_Disc_D8.0mm_W5.0mm_P5.00mm" H 7988 3600 50  0001 C CNN
 F 3 "~" H 7950 3750 50  0001 C CNN
 	1    7950 3750
@@
 F 0 "R7" V 7257 2500 50  0000 C CNN
 F 1 "100" V 7166 2500 50  0000 C CNN
-F 2 "Resistor_THT:R_Axial_DIN0309_L9.0mm_D3.2mm_P15.24mm_Horizontal" V 6980 2500 50  0001 C CNN
+F 2 "Resistor_THT:R_Axial_DIN0207_L6.3mm_D2.5mm_P10.16mm_Horizontal" V 6980 2500 50  0001 C CNN
 F 3 "~" H 7050 2500 50  0001 C CNN
 	1    7050 2500
@@
 F 0 "R8" H 7020 5296 50  0000 L CNN
 F 1 "100" H 7020 5205 50  0000 L CNN
-F 2 "Resistor_THT:R_Axial_DIN0309_L9.0mm_D3.2mm_P15.24mm_Horizontal" V 6880 5250 50  0001 C CNN
+F 2 "Resistor_THT:R_Axial_DIN0207_L6.3mm_D2.5mm_P10.16mm_Horizontal" V 6880 5250 50  0001 C CNN
 F 3 "~" H 6950 5250 50  0001 C CNN
 	1    6950 5250
@@
 Wire Wire Line
 	6000 3950 6000 4150
-Text Notes 5550 3550 0    50   ~ 0
+Text Notes 4950 3600 0    50   ~ 0
 Gain Adjust
 Wire Wire Line
